Commit message: [EDIT] xacro file
- LiDAR Sensor 추가하기 위해 Xacro 파일 수정했음
- /로 인한 충돌이 있어 drone.yaml 파일의 namespace 수정
- rviz 파일에 LaserScan 추가했음

File: sjtu_drone_description/urdf/sjtu_drone.urdf.xacro (robot description, xacro)
@@ -54,4 +54,22 @@
   </joint>
   <link name="bottom_cam_link"/>
+  <joint name="lidar_joint" type="fixed">
+    <parent link="base_link" />
+    <child link="lidar_link" />
+    <origin rpy="0 0 0" xyz="0 0 0"/>
+  </joint>
+  <link name="lidar_link">
+    <visual>
+            <geometry>
+                <cylinder radius="0.03" length="0.03"/>
+            </geometry>
+            <material name="red"/>
+      </visual>
+      <collision>
+          <geometry>
+              <cylinder radius="0.03" length="0.03"/>
+          </geometry>
+      </collision>
+  </link>
   <gazebo>
     <plugin name='simple_drone' filename='libplugin_drone.so'>
@@ -284,3 +302,31 @@
     </sensor>
   </gazebo>
+  <gazebo reference="lidar_link">
+    <sensor name="laser" type="ray">
+      <always_on>1</always_on>
+      <visualize>1</visualize>
+      <update_rate>10</update_rate>
+      <ray>
+        <scan>
+          <horizontal>
+            <samples>360</samples>
+            <resolution>1.000000</resolution>
+            <min_angle>-3.14</min_angle>
+            <max_angle>3.14</max_angle>
+          </horizontal>
+        </scan>
+        <range>
+          <min>0.2</min>
+          <max>10</max>
+        </range>
+      </ray>
+      <plugin name="laser_controller" filename="libgazebo_ros_ray_sensor.so">
+        <ros>
+          <namespace>${mp['namespace']}</namespace>
+        </ros>
+        <frame_name>${mp['namespace']}/lidar_link</frame_name>
+        <output_type>sensor_msgs/LaserScan</output_type>
+      </plugin>
+    </sensor>
+  </gazebo>
 </robot>

Commit message: [EDIT] Xacro
- Add Bottom 3D LiDAR

File: sjtu_drone_description/urdf/sjtu_drone.urdf.xacro (robot description, xacro)
@@ -36,10 +36,10 @@
     </visual>
   </link>
-  <joint name="sonar_joint" type="fixed">
+  <joint name="bottom_lidar_joint" type="fixed">
     <parent link="base_link" />
-    <child link="sonar_link" />
-    <origin rpy="0 ${M_PI/2} 0" xyz="0 0 0"/>
-  </joint>
-  <link name="sonar_link"/>
+    <child link="bottom_lidar_link" />
+    <origin rpy="0 0 0" xyz="0 0 0"/>
+  </joint>
+  <link name="bottom_lidar_link"/>
   <joint name="front_cam_joint" type="fixed">
     <origin rpy="0 0 0" xyz="0.2 0 0"/>
@@ -59,17 +59,5 @@
     <origin rpy="0 0 0" xyz="0 0 0"/>
   </joint>
-  <link name="lidar_link">
-    <visual>
-            <geometry>
-                <cylinder radius="0.03" length="0.03"/>
-            </geometry>
-            <material name="red"/>
-      </visual>
-      <collision>
-          <geometry>
-              <cylinder radius="0.03" length="0.03"/>
-          </geometry>
-      </collision>
-  </link>
+  <link name="lidar_link"/>
   <gazebo>
     <plugin name='simple_drone' filename='libplugin_drone.so'>
@@ -145,44 +133,35 @@
     </sensor>
   </gazebo>
-  <!-- Sonar sensor in 100fps -->
-  <gazebo reference="sonar_link">
-    <sensor name="sonar" type="ray">
-      <always_on>1</always_on>
-      <visualize>1</visualize>
-      <update_rate>30</update_rate>
+  <gazebo reference="bottom_lidar_link">
+    <sensor name="laser" type="ray">
+      <always_on>1</always_on>
+      <visualize>1</visualize>
+      <update_rate>60</update_rate>
       <ray>
         <scan>
           <horizontal>
-            <samples>5</samples>
+            <samples>360</samples>
             <resolution>1.000000</resolution>
-            <min_angle>-0.12</min_angle>
-            <max_angle>0.12</max_angle>
+            <min_angle>-3.14</min_angle>
+            <max_angle>3.14</max_angle>
           </horizontal>
           <vertical>
-            <samples>5</samples>
+            <samples>50</samples>
             <resolution>1.000000</resolution>
-            <min_angle>-0.12</min_angle>
-            <max_angle>0.12</max_angle>
+            <min_angle>-3.14</min_angle>
+            <max_angle>0</max_angle>
           </vertical>
         </scan>
         <range>
-          <min>0.02</min>
-          <max>10</max>
-          <resolution>0.01</resolution>
+          <min>0.2</min>
+          <max>3</max>
         </range>
-        <noise>
-          <type>gaussian</type>
-          <mean>0.0</mean>
-          <stddev>0.01</stddev>
-        </noise>
       </ray>
-      <plugin name="sonar" filename="libgazebo_ros_ray_sensor.so">
-        <ros>
-          <namespace>${mp['namespace']}</namespace>
-          <!-- <remapping>~/out:=sonar</remapping> -->
-        </ros>
-        <frame_name>${mp['namespace']}/sonar_link</frame_name>
-        <output_type>sensor_msgs/Range</output_type>
-        <radiation_type>ultrasound</radiation_type>
+      <plugin name="bottome_laser_controller" filename="libgazebo_ros_ray_sensor.so">
+        <ros>
+          <namespace>${mp['namespace']}</namespace>
+        </ros>
+        <frame_name>${mp['namespace']}/bottom_lidar_link</frame_name>
+        <output_type>sensor_msgs/PointCloud2</output_type>
       </plugin>
     </sensor>
@@ -306,5 +285,5 @@
       <always_on>1</always_on>
       <visualize>1</visualize>
-      <update_rate>10</update_rate>
+      <update_rate>60</update_rate>
       <ray>
         <scan>

Commit message: 성능 개선 / 함수 수정

File: sjtu_drone_description/urdf/sjtu_drone.urdf.xacro (robot description, xacro)
@@ -36,10 +36,4 @@
     </visual>
   </link>
-  <joint name="bottom_lidar_joint" type="fixed">
-    <parent link="base_link" />
-    <child link="bottom_lidar_link" />
-    <origin rpy="0 0 0" xyz="0 0 0"/>
-  </joint>
-  <link name="bottom_lidar_link"/>
   <joint name="front_cam_joint" type="fixed">
     <origin rpy="0 0 0" xyz="0.2 0 0"/>
@@ -133,39 +127,4 @@
     </sensor>
   </gazebo>
-  <gazebo reference="bottom_lidar_link">
-    <sensor name="bottom_laser" type="ray">
-      <always_on>1</always_on>
-      <visualize>1</visualize>
-      <update_rate>60</update_rate>
-      <ray>
-        <scan>
-          <horizontal>
-            <samples>360</samples>
-            <resolution>1.000000</resolution>
-            <min_angle>-3.14</min_angle>
-            <max_angle>3.14</max_angle>
-          </horizontal>
-          <vertical>
-            <samples>80</samples>
-            <resolution>1.000000</resolution>
-            <min_angle>-3.14</min_angle>
-            <max_angle>-1</max_angle>
-          </vertical>
-        </scan>
-        <range>
-          <min>0.2</min>
-          <max>3</max>
-        </range>
-      </ray>
-      <plugin name="bottome_laser_controller" filename="libgazebo_ros_ray_sensor.so">
-        <ros>
-          <namespace>${mp['namespace']}</namespace>
-          <remapping>~/out:=bottom_lidar</remapping>
-        </ros>
-        <frame_name>${mp['namespace']}/bottom_lidar_link</frame_name>
-        <output_type>sensor_msgs/PointCloud2</output_type>
-      </plugin>
-    </sensor>
-  </gazebo>
   <gazebo reference="front_cam_link">
     <sensor name="front_camera" type="camera">
